File: E0001_fader_driver.kicad_sch (KiCad schematic)
At the start: 34 parts, among them J1 JST GH SM04B-GHS-TB, J2 TC2030-IDC-NL, Q1 AO3401A, U1 STM32C051F6P6, U2 MCP1703A-3302E/CB, U3 DRV8210PDSGR

Commit message: E0001 rev C: PBUS v2 input, local eFuse, UART bootloader header, fab outputs
- Supply from E0003 peripheral bus v2 (PBUS 6-9 V) instead of 5 V
- TPS259470A local eFuse (OVLO, 0.6 A limit, reverse blocking); SMF9.0A after eFuse
- MCP1703A SOT-89 LDO; DRV8210 logic on 3V3
- Tag-Connect SWD replaced by 1x6 right-angle UART bootloader header (J2)
- No test points; common cross-project parts; PBUS 6-9 V silkscreen
- Rev B archived in archive/revB; fab outputs in fab/E0001_revB and fab/E0001_revC
- Spec docs/SPEC_revC.md v1.0, schematic notes, layout review r1 (PASS)

Co-Authored-By: Claude Opus 5.5 <noreply@anthropic.com>
Parts:
- removed Q1: AO3401A, Package_TO_SOT_SMD:SOT-23, symbol Transistor_FET:AO3401A
- removed R1: 10k, Resistor_SMD:R_0402_1005Metric, symbol Device:R_Small_US
- added C15: 4.7nF, Capacitor_SMD:C_0402_1005Metric, symbol Device:C_Small
- added C16: 1.8nF, Capacitor_SMD:C_0402_1005Metric, symbol Device:C_Small
- added C17: 100nF, Capacitor_SMD:C_0402_1005Metric, symbol Device:C_Small
- added C18: 4.7uF, Capacitor_SMD:C_0603_1608Metric, symbol Device:C_Small
- added C19: 1nF, Capacitor_SMD:C_0402_1005Metric, symbol Device:C_Small
- added C20: 10uF, Capacitor_SMD:C_0805_2012Metric, symbol Device:C_Small
- added D4, D5: PESD5V0L1UL, Diode_SMD:D_SOD-882, symbol Diode:PESD5V0L1UL
- added D6, D7: BAT54W, Package_TO_SOT_SMD:SOT-323_SC-70, symbol Diode:BAT54W
- added R11, R13: 1M 1%, Resistor_SMD:R_0402_1005Metric, symbol Device:R_Small_US
- added R12: 330k 1%, Resistor_SMD:R_0402_1005Metric, symbol Device:R_Small_US
- added R14: 137k 1%, Resistor_SMD:R_0402_1005Metric, symbol Device:R_Small_US
- added R15: 5.23k 1%, Resistor_SMD:R_0402_1005Metric, symbol Device:R_Small_US
- added R16, R17: 10k, Resistor_SMD:R_0402_1005Metric, symbol Device:R_Small_US
- added R18: 1k, Resistor_SMD:R_0402_1005Metric, symbol Device:R_Small_US
- added R19, R20: 0R, Resistor_SMD:R_0402_1005Metric, symbol Device:R_Small_US
- added U4: TPS259470ARPW, E0001:TI_RPW0010A_VQFN-HR-10_2x2mm_P0.475mm, symbol E0001:TPS259470L
- C1: Dielectric X5R -> (none); DigiKey 1276-2402-1-ND -> (none); MPN CL21A106KPCLQNC -> TMK212BBJ106MG-T; Manufacturer Samsung -> Taiyo Yuden; Supplier (none) -> DigiKey; Supplier PN (none) -> 587-6025-1-ND; Voltage 10V -> 25V
- C10, C13, C4, C6, C7, C9: DigiKey 1276-1505-1-ND -> (none); MPN CL05B104JO5NNNC -> GRM155R71H104KE14D; Manufacturer Samsung -> Murata Electronics; Supplier (none) -> DigiKey; Supplier PN (none) -> 490-10700-1-ND; Voltage (none) -> 50V
- C11, C12: value 22uF -> 10uF; Dielectric X5R -> (none); MPN CL21A226MOQNNNE -> TMK212BBJ106MG-T; Manufacturer Samsung -> Taiyo Yuden; Supplier (none) -> DigiKey; Supplier PN (none) -> 587-6025-1-ND; Voltage 10V -> 25V
- C14: Manufacturer Murata -> Murata Electronics; Supplier (none) -> DigiKey; Supplier PN (none) -> 490-4516-1-ND; Voltage (none) -> 50V
- C2, C5: Dielectric X5R -> (none); DigiKey 490-7203-1-ND -> (none); Manufacturer Murata -> Murata Electronics; Supplier (none) -> DigiKey; Supplier PN (none) -> 490-7203-1-ND; Voltage 10V -> 25V
- C3: Dielectric X5R -> (none); DigiKey 1276-1076-1-ND -> (none); Manufacturer Samsung -> Samsung Electro-Mechanics; Supplier (none) -> DigiKey; Supplier PN (none) -> 1276-1076-1-ND; Voltage 10V -> (none)
- D1: value SMF5V0A -> SMF9.0A; footprint Diode_SMD:D_SMF -> Diode_SMD:D_SOD-123F; symbol Diode:SMF5V0A -> Diode:SMF9V0A; DigiKey F5748CT-ND -> (none); MPN SMF5.0A -> SMF9.0A; Manufacturer Littelfuse -> Littelfuse Inc.; Supplier (none) -> DigiKey; Supplier PN (none) -> F5755CT-ND
- D2: DigiKey 1727-4193-1-ND -> (none); Manufacturer Nexperia -> Nexperia USA Inc.; Supplier (none) -> DigiKey; Supplier PN (none) -> 1727-4193-1-ND
- D3: DigiKey 160-1446-1-ND -> (none); Manufacturer Lite-On -> Lite-On Inc.; Supplier (none) -> DigiKey; Supplier PN (none) -> 160-1446-1-ND
- J1: value JST GH SM04B-GHS-TB -> SM04B-GHS-TB; Manufacturer JST -> JST Sales America Inc.; Supplier (none) -> LCSC; Supplier PN (none) -> LCSC C189895 (SM04B-GHS-TB(LF)(SN))
- J2: value TC2030-IDC-NL -> 61300611021; footprint Connector:Tag-Connect_TC2030-IDC-NL_2x03_P1.27mm_Vertical -> Connector_PinHeader_2.54mm:PinHeader_1x06_P2.54mm_Horizontal; symbol Connector:Conn_ARM_SWD_TagConnect_TC2030 -> Connector_Generic:Conn_01x06; MPN (none) -> 61300611021; Manufacturer (none) -> Würth Elektronik; Supplier (none) -> DigiKey; Supplier PN (none) -> 732-5339-ND; now in the parts list
- R10, R7: DigiKey 311-1.00KLRCT-ND -> (none); Manufacturer Yageo -> YAGEO; Supplier (none) -> DigiKey; Supplier PN (none) -> 311-1.00KLRCT-ND
- R2: DigiKey 311-10.0HRCT-ND -> (none); Manufacturer Yageo -> YAGEO; Supplier (none) -> DigiKey; Supplier PN (none) -> 311-10.0HRCT-ND
- R5: DigiKey 311-4.7KLRCT-ND -> (none); MPN RC0402FR-074K7L -> RK73H1ETTP4701F; Manufacturer Yageo -> KOA Speer Electronics, Inc.; Supplier (none) -> DigiKey; Supplier PN (none) -> 2019-RK73H1ETTP4701FCT-ND
- R6: DigiKey 311-1.00MLRCT-ND -> (none); Manufacturer Yageo -> YAGEO; Supplier (none) -> DigiKey; Supplier PN (none) -> 311-1.00MLRCT-ND
- R8: DigiKey 311-100KLRCT-ND -> (none); Manufacturer Yageo -> YAGEO; Supplier (none) -> DigiKey; Supplier PN (none) -> 311-100KLRCT-ND
- R9: value 100k -> 30.1k 1%; DigiKey 311-100KLRCT-ND -> (none); MPN RC0402FR-07100KL -> RC0402FR-0730K1L; Manufacturer Yageo -> YAGEO; Supplier (none) -> DigiKey; Supplier PN (none) -> 311-30.1KLRCT-ND
- RV1: MPN (none) -> RSA0N11M9A0J B10K clone; Manufacturer (none) -> Fastigeaty (seller Fadianshop); Supplier (none) -> Amazon.de; Supplier PN (none) -> ASIN B0H45B29YK
- U1: DigiKey 497-STM32C051F6P6-ND -> (none); Supplier (none) -> DigiKey; Supplier PN (none) -> 497-STM32C051F6P6-ND
- U2: value MCP1703A-3302E/CB -> MCP1703AT-3302E/MB; footprint Package_TO_SOT_SMD:SOT-23 -> Package_TO_SOT_SMD:SOT-89-3; symbol Regulator_Linear:MCP1703Ax-330xxTT -> Regulator_Linear:MCP1703Ax-330xxMB; DigiKey MCP1703AT-3302E/CBCT-ND -> (none); MPN MCP1703AT-3302E/CB -> MCP1703AT-3302E/MB; Manufacturer Microchip -> Microchip Technology; Supplier (none) -> DigiKey; Supplier PN (none) -> MCP1703AT-3302E/MBCT-ND
- U3: DigiKey 296-DRV8210PDSGRCT-ND -> (none); Supplier (none) -> DigiKey; Supplier PN (none) -> 296-DRV8210PDSGRCT-ND
Connections:
- net +3V3: now also C10.1, RV1.3 (END_TOP), U2.3 (VO), U3.8 (VCC); no longer J2.1 (VCC), U2.2 (VO)
- net ADDR0: now also U1.18 (PA13); no longer U1.16 (PA9/PA11)
- net ADDR1: now also U1.3 (PC15); no longer U1.17 (PA10/PA12)
- net GND: now also J2.1 (Pin_1), C15.2, C16.2, C17.2, C18.2, C19.2, C20.2, D4.2 (A), D5.2 (A), R12.2, R14.2, R15.2, R17.2, U4.8 (GND); no longer J2.5 (GND)
- net I2C_SCL: now also R19.2; no longer J1.2 (Pin_2)
- net I2C_SDA: now also R20.2; no longer J1.3 (Pin_3)
- net LDO_IN: now also U2.2 (VI), D7.3 (K); no longer U2.3 (VI)
- net NRST: now also D6.1 (A); no longer J2.3 (~{RESET})
- net J2_NRST: now reaches J2.6 (Pin_6)
- net J2_NRST: now also D6.3 (K)
- net +5V renamed VM_P
- net VM_P: now also C20.1, U4.6 (OUT); no longer C10.1, U3.8 (VCC)
- net POT_HI renamed ILM_ADC
- net ILM_ADC: now also C19.1, R16.2; no longer RV1.3 (END_TOP)
- net SWCLK renamed BOOT0
- net BOOT0: now also R17.1, R18.2; no longer J2.4 (SWCLK)
- net SWDIO renamed J2_3V3
- net J2_3V3: now also D7.1 (A); no longer U1.18 (PA13)
- net VIN renamed PBUS_IN
- net PBUS_IN: now also C17.1, C18.1, R11.1, R13.1, U4.5 (IN)
- new net EF_DVDT: C16.1, U4.7 (DVDT)
- new net EF_EN: R11.2, R12.1, U4.1 (EN/UVLO)
- new net EF_ILM: R15.1, R16.1, U4.9 (ILM)
- new net EF_ITIMER: C15.1, U4.10 (ITIMER)
- new net EF_OVLO: R13.2, R14.1, U4.2 (OVLO)
- new net J1_SCL: D4.1 (K), J1.2 (Pin_2), R19.1
- new net J1_SDA: D5.1 (K), J1.3 (Pin_3), R20.1
- new net J2_BOOT0: J2.5 (Pin_5), R18.1
- new net UART_RX: J2.3 (Pin_3), U1.17 (PA10/PA12)
- new net UART_TX: J2.4 (Pin_4), U1.16 (PA9/PA11)
- no-connect marks 2 -> 4
Other:
- note added: "ADDRn = 1 when its jumper is open (internal pull-up)."
- note added: "Auto-boot: B0 high, pulse RST low, release."
- note added: "C4 at VDD (C3/C5 at the LDO). C6: NRST filter."
- note added: "FADER RV1: TRACK, TOUCH, MOTOR"
- note added: "HOST J1 (PBUS v2 + I2C), eFUSE U4 TPS259470A"
- note added: "I2C address jumpers (bottom): open = 1"
- note added: "ILM monitor 0.95 V/A -> R16 10k + C19 1 nF -> PA2. FLT and AUXOFF unused."
- note added: "ITIMER 4.7 nF ~3.9 ms, dVdt 1.8 nF ~1.1 V/ms. Reverse blocking to -15 V, survives 11 V (OVLO off)."
- note added: "J1: 1 PBUS 2 SCL 3 SDA 4 GND, MP = GND. Silk "PBUS 6-9 V"."
- note added: "J2 UART BOOTLOADER HEADER (1x6 2.54 R/A)"
- note added: "J2 pin 2 (3V3) feeds LDO_IN through D7 BAT54W, so VOUT never exceeds VIN (MCP1703A abs max)."
- note added: "MCU STM32C051F6P6 (TSSOP-20)"
- note added: "MOTOR DRIVER DRV8210P"
- note added: "No I2C pull-ups here (host 4.7k). R19/R20 0R (<= 100R allowed)."
- note added: "Option bytes at first flash: nBOOT_SEL=0,"
- note added: "PA11/PA12/PA15/PB3-5/PB8 (bonded) stay inputs."
- note added: "Pin 2: adapter 3V3 -> D7 -> LDO_IN (board ~2.9 V)."
- note added: "Pin 5: R18 1k series, R17 10k pull-down at PA14."
- note added: "Pin 6: D6 lets the adapter only pull NRST low."
- note added: "Pins 16/17 = PA9/PA10 USART1 (ROM bootloader TX/RX),"
- note added: "Silk: GND 3V3 RX TX B0 RST, "UART boot 3.3 V"."
- note added: "Touch: T -> D2, R5 -> PA0; R6 1M from PA1."
- note added: "Track top -> +3V3 (rev C), wiper R7/C7 -> PA3."
- note added: "U4 TPS259470A (auto-retry): UVLO 4.84/4.40 V, OVLO 9.96/9.05 V, I_LIM 3334/5.23k = 0.64 A (0.54-0.73 A),"
- note added: "VM = VM_P (<= 9 V), VCC = +3V3. C14 DNP."
- note added: "VM_P (protected PBUS), PBUS SENSE, 3V3 LDO"
- note added: "VM_P bulk 4 x 10 uF 25 V (~45 uF total input incl. C18). D1 SMF9.0A clamps back-EMF on VM_P."
- note added: "VSENSE = VM_P x 30.1/130.1 -> PA4 (11 V -> 2.55 V). U2 MCP1703A SOT-89 from VM_P via R2 10R."
- note added: "nBOOT1=1, BOOT_LOCK=0. No SWD, no test points."
- note added: "pin 19 = PA14-BOOT0 (R17 10k pull-down). Address 0x30 | ADDR,"
- note removed: "(2.2k-4.7k to the bus logic level; SDA/SCL"
- note removed: "10R + 4.7uF: keeps motor PWM"
- note removed: "3.3 V LDO"
- note removed: "C13 = VCC, C10-C12 = VM decoupling. C14 not fitted (brush-noise option)."
- note removed: "End 1 (bottom of travel) = GND, so FADER_POS rises toward the top."
- note removed: "FADER: POSITION, TOUCH, MOTOR (ALPS RSA0N11M9A0J)"
- note removed: "FG = fader frame lugs: soldered for retention, tied to GND."
- note removed: "I2C address select:"
- note removed: "I2C pull-ups: on the host side"
- note removed: "IN1 = PWM, IN2 = 0: knob moves down. IN1 = IN2 = 1: brake."
- note removed: "IN2 = PWM, IN1 = 0: M+ positive, knob moves to the top of travel (ALPS)."
- note removed: "J1: JST GH 1.25 mm, Dronecode/Pixhawk I2C pinout: 1 = +5 V, 2 = SCL, 3 = SDA, 4 = GND"
- note removed: "MCP1703A: 16 V max in, 2 uA Iq"
- note removed: "MCU STM32C051F6P6"
- note removed: "MOTOR DRIVER (DRV8210P, DRV8837-compatible, motor from +5 V)"
- note removed: "POWER INPUT, PROTECTION, SUPPLY SENSE"
- note removed: "Position: track powered from POT_HI (PA2 high), wiper read on PA3 (ratiometric)."
- note removed: "SWD (Tag-Connect TC2030-NL pads)"
- note removed: "Status LED"
- note removed: "TIM2 capture on PA0) or by ADC charge sharing on PA0."
- note removed: "Touch: conductive knob -> lever -> T. Sense by RC charge time (PA1 drives via 1M,"
- note removed: "VSENSE = +5 V / 2 (PA4)"
- note removed: "open = 1, bridged = 0"
- note removed: "pins are 5 V tolerant, 3.3 V or 5 V bus OK)"
- note removed: "ripple out of the LDO."
- moved on the sheet: C1, C10, C11, C12, C13, C14, C2, C3, C4, C5, C6, C7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
